File: pcb/ci-84.kicad_sch (KiCad schematic)
At the start: 124 parts, among them J1 jst-battery, SW1 SW_Push, SW10 XT0N, SW11 STAT, SW12 MATH, SW13 APPS, SW14 PRGM, SW15 VARS, SW16 CLEAR, SW17 X^-1, SW18 SIN, SW19 COS, SW2 Y=, SW20 TAN, SW21 ^, SW22 X^2, SW23 ,, SW24 (, SW25 ), SW26 DIVIDE, SW27 LOG, SW28 7, SW29 8, SW3 WINDOW, SW30 9, SW31 MULITPLY, SW32 IN, SW33 4, SW34 5, SW35 6, SW36 SUBTRACT, SW37 STO, SW38 1, SW39 2, SW4 ZOOM, SW40 3, SW41 ADD, SW42 ON, SW43 0, SW44 ., SW45 (-), SW46 ENTER, SW47 GRAPH, SW48 UP, SW49 RIGHT, SW5 TRACE, SW50 DOWN, SW51 LEFT, SW6 2ND, SW7 MODE, SW8 DEL, SW9 ALPHA, U1 STM32L471RGTx, U3 TPS63900, U4 TFT_320x240

Commit message: sw pins
Connections:
- net IO_DC: now also U1.45 (PA12); no longer U1.49 (PA14)
- net SWDIO: now reaches U1.46 (PA13)
- new net SWCLK: U1.49 (PA14)
Changed lines of the file:
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@@
+		)
+	)
+	(label "SWCLK"
+		(at 90.17 143.51 0)
+		(effects
+			(font
+				(size 1.27 1.27)
+			)
+			(justify left bottom)
 		)
 	)
@@
 		)
 	)
+	(label "SWDIO"
+		(at 90.17 140.97 0)
+		(effects
+			(font
+				(size 1.27 1.27)
+			)
+			(justify left bottom)
+		)
+	)
 	(label "c4"
 		(at 54.61 168.91 180)
@@
 	)
 	(label "IO_DC"
-		(at 90.17 143.51 0)
-		(effects
-			(font
+		(at 90.17 138.43 0)
+		(effects
+			(font

Commit message: swd
Parts:
- added J2: SWD, Connector_PinHeader_2.54mm:PinHeader_1x04_P2.54mm_Vertical, symbol Connector_Generic:Conn_01x04
Connections:
- net GND: now also J2.2 (Pin_2)
- net SWCLK: now also J2.3 (Pin_3)
- net SWDIO: now also J2.4 (Pin_4)
- net VDD: now also J2.1 (Pin_1)
Other:
- moved on the sheet: C11, C12, L1, R5, U3, U4

Commit message: cleaned schematic and added final components
Parts:
- BT1: footprint (none) -> Battery:BatteryHolder_MPD_BC2003_1x2032
- L1: footprint (none) -> Inductor_SMD:L_1008_2520Metric
- R1, R2, R3, R4, R5: footprint (none) -> Resistor_SMD:R_0603_1608Metric
Connections:
- net GND: now also BT1.2 (-)
- net VBAT: now reaches BT1.1 (+)
- net VBAT: now also U1.1 (VBAT)
- no-connect marks 0 -> 22
Other:
- removed sheet Keyboard Matrix
- removed sheet Screen
- removed sheet Voltage Regulator
- removed sheet stm32
- note added: "Keyboard Matrix"
- note added: "STM32"
- note added: "Screen"
- note added: "Voltage Regulator"
